File: driver.kicad_sch (KiCad schematic)
At the start: 6 parts, among them J1 Conn_01x03, J2 Conn_01x03, J3 Conn_01x03

Commit message: adding missing pullups
Parts:
- added R1 (x2): 3k3, Resistor_SMD:R_1206_3216Metric, symbol Device:R
Connections:
- net 5v: now also R1.2, R1.2
- net dir: now also R1.1
- net step: now also R1.1
Changed lines of the file:
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@@
+    (stroke (width 0) (type default))
+  )
+  (wire (pts (xy 59.69 62.23) (xy 59.69 69.85))
     (stroke (width 0) (type default))
   )
@@
     )
   )
+  (global_label "5v" (shape input) (at 59.69 62.23 0) (fields_autoplaced)
+    (effects (font (size 1.27 1.27)) (justify left))
+    (property "Intersheetrefs" "${INTERSHEET_REFS}" (at 64.7729 62.23 0)
+      (effects (font (size 1.27 1.27)) (justify left) hide)
+    )
+  )
   (global_label "5v" (shape input) (at 64.77 77.47 180) (fields_autoplaced)
     (effects (font (size 1.27 1.27)) (justify right))
@@
     )
   )
+  (hierarchical_label "dir" (shape input) (at 52.07 69.85 180) (fields_autoplaced)
+    (effects (font (size 1.27 1.27)) (justify right))
+  )
   (hierarchical_label "dir" (shape input) (at 96.52 72.39 180) (fields_autoplaced)
     (effects (font (size 1.27 1.27)) (justify right))
@@
   )
   (hierarchical_label "step" (shape input) (at 96.52 69.85 180) (fields_autoplaced)
+    (effects (font (size 1.27 1.27)) (justify right))
+  )
+  (hierarchical_label "step" (shape input) (at 52.07 62.23 180) (fields_autoplaced)
     (effects (font (size 1.27 1.27)) (justify right))
   )
@@
     )
   )
+  (symbol (lib_id "Device:R") (at 55.88 62.23 90) (unit 1)
+    (in_bom yes) (on_board yes) (dnp no)
+    (property "Reference" "R1" (at 55.88 59.69 90)
+      (effects (font (size 1.27 1.27)))
+    )
+    (property "Value" "3k3" (at 55.88 64.77 90)
+      (effects (font (size 1.27 1.27)))
+    )
+    (property "Footprint" "Resistor_SMD:R_1206_3216Metric" (at 55.88 64.008 90)
+      (effects (font (size 1.27 1.27)) hide)
+    )
+    (property "Datasheet" "~" (at 55.88 62.23 0)
+      (effects (font (size 1.27 1.27)) hide)
+    )
+    (pin "1")
+    (pin "2")
+    (instances
+      (project "riowerks"
+        (path "/c4675d0b-5c1c-444a-a1ef-26bf66f46aa5/cda04744-3ce8-4a6b-a82d-a1325fcc2daa"
+          (reference "R1") (unit 1)
+        )
+        (path "/c4675d0b-5c1c-444a-a1ef-26bf66f46aa5/c87ea30f-b16d-4690-be9f-7e9196f340db"
+          (reference "R2") (unit 1)
+        )
+        (path "/c4675d0b-5c1c-444a-a1ef-26bf66f46aa5/0caef072-d6e6-4191-8609-a2a060f30d09"
+          (reference "R3") (unit 1)
+        )
+        (path "/c4675d0b-5c1c-444a-a1ef-26bf66f46aa5/9b7eb7c2-dba6-4078-aea0-2fd449da534f"
+          (reference "R4") (unit 1)
+        )
+        (path "/c4675d0b-5c1c-444a-a1ef-26bf66f46aa5/c4b53cc4-45b0-40c6-a2e4-f85052d4ed8a"
+          (reference "R5") (unit 1)
+        )
+        (path "/c4675d0b-5c1c-444a-a1ef-26bf66f46aa5/6dac5bea-3ac5-4905-a711-17de9963fb48"
+          (reference "R6") (unit 1)
+        )
+        (path "/c4675d0b-5c1c-444a-a1ef-26bf66f46aa5/0e9d2bbf-2b0b-4860-a06b-304bc4546dd9"
+          (reference "R7") (unit 1)
+        )
+        (path "/c4675d0b-5c1c-444a-a1ef-26bf66f46aa5/77b70234-a638-4cba-af0b-c8e26a05632f"
+          (reference "R8") (unit 1)
+        )
+        (path "/c4675d0b-5c1c-444a-a1ef-26bf66f46aa5/341fad45-713c-4626-966f-e3afd8f08c91"
+          (reference "R16") (unit 1)
+        )
+        (path "/c4675d0b-5c1c-444a-a1ef-26bf66f46aa5"
+          (reference "R43") (unit 1)
+        )
+      )
+      (project "rio-icebreaker3x"
+        (path "/cfe43c71-4742-4fe7-be75-9d9a9d4efd01"
+          (reference "R5") (unit 1)
+        )
+        (path "/cfe43c71-4742-4fe7-be75-9d9a9d4efd01/01713ad6-c8ee-4cb4-a069-0eb1e2d0d4c5"
+          (reference "R15") (unit 1)
+        )
+        (path "/cfe43c71-4742-4fe7-be75-9d9a9d4efd01/71bd7516-8b6e-4c0f-97ca-5abb746077c1"
+          (reference "R16") (unit 1)
+        )
+        (path "/cfe43c71-4742-4fe7-be75-9d9a9d4efd01/d8c46525-3323-49c5-8ba1-282344862c7d"
+          (reference "R17") (unit 1)
+        )
+      )
+    )
+  )
   (symbol (lib_id "Connector_Generic:Conn_01x03") (at 91.44 80.01 180) (unit 1)
     (in_bom yes) (on_board yes) (dnp no)
@@
         )
       )
+    )
+  )
+  (symbol (lib_id "Device:R") (at 55.88 69.85 90) (unit 1)
+    (in_bom yes) (on_board yes) (dnp no)
+    (property "Reference" "R1" (at 55.88 67.31 90)
+      (effects (font (size 1.27 1.27)))
+    )
+    (property "Value" "3k3" (at 55.88 72.39 90)
+      (effects (font (size 1.27 1.27)))
+    )
+    (property "Footprint" "Resistor_SMD:R_1206_3216Metric" (at 55.88 71.628 90)
+      (effects (font (size 1.27 1.27)) hide)
+    )
+    (property "Datasheet" "~" (at 55.88 69.85 0)
+      (effects (font (size 1.27 1.27)) hide)
+    )
+    (pin "1")
+    (pin "2")
+    (instances
+      (project "riowerks"
+        (path "/c4675d0b-5c1c-444a-a1ef-26bf66f46aa5/cda04744-3ce8-4a6b-a82d-a1325fcc2daa"
+          (reference "R1") (unit 1)
+        )
+        (path "/c4675d0b-5c1c-444a-a1ef-26bf66f46aa5/c87ea30f-b16d-4690-be9f-7e9196f340db"
+          (reference "R2") (unit 1)
+        )
+        (path "/c4675d0b-5c1c-444a-a1ef-26bf66f46aa5/0caef072-d6e6-4191-8609-a2a060f30d09"
+          (reference "R3") (unit 1)
+        )
+        (path "/c4675d0b-5c1c-444a-a1ef-26bf66f46aa5/9b7eb7c2-dba6-4078-aea0-2fd449da534f"
+          (reference "R4") (unit 1)
+        )
+        (path "/c4675d0b-5c1c-444a-a1ef-26bf66f46aa5/c4b53cc4-45b0-40c6-a2e4-f85052d4ed8a"
+          (reference "R5") (unit 1)
+        )
+        (path "/c4675d0b-5c1c-444a-a1ef-26bf66f46aa5/6dac5bea-3ac5-4905-a711-17de9963fb48"
+          (reference "R6") (unit 1)
+        )
+        (path "/c4675d0b-5c1c-444a-a1ef-26bf66f46aa5/0e9d2bbf-2b0b-4860-a06b-304bc4546dd9"
+          (reference "R7") (unit 1)
+        )
+        (path "/c4675d0b-5c1c-444a-a1ef-26bf66f46aa5/77b70234-a638-4cba-af0b-c8e26a05632f"
+          (reference "R8") (unit 1)
+        )
+        (path "/c4675d0b-5c1c-444a-a1ef-26bf66f46aa5/341fad45-713c-4626-966f-e3afd8f08c91"
+          (reference "R16") (unit 1)
+        )
+        (path "/c4675d0b-5c1c-444a-a1ef-26bf66f46aa5"
+          (reference "R43") (unit 1)
+        )
+      )
+      (project "rio-icebreaker3x"
+        (path "/cfe43c71-4742-4fe7-be75-9d9a9d4efd01"
+          (reference "R5") (unit 1)
+        )
+        (path "/cfe43c71-4742-4fe7-be75-9d9a9d4efd01/01713ad6-c8ee-4cb4-a069-0eb1e2d0d4c5"
+          (reference "R7") (unit 1)
+        )
+        (path "/cfe43c71-4742-4fe7-be75-9d9a9d4efd01/71bd7516-8b6e-4c0f-97ca-5abb746077c1"
+          (reference "R8") (unit 1)
+        )
+        (path "/cfe43c71-4742-4fe7-be75-9d9a9d4efd01/d8c46525-3323-49c5-8ba1-282344862c7d"
+          (reference "R9") (unit 1)
+        )
+      )
