File: rio-icebreaker3x.kicad_pcb (KiCad board)
At the start: 2 copper layers, 78.7 x 51.9 mm, 53 parts, among them J1 Conn_01x03, J10 Conn_01x03, J11 Conn_01x03, J15 Conn_02x06_Odd_Even, J16 Conn_02x06_Odd_Even, J2 Conn_01x03, J3 Conn_01x03, J4 Conn_01x03, J5 Conn_01x03, J6 Conn_01x03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

Commit message: adding missing pullups
Parts:
- added R15: 3k3, Resistor_SMD:R_1206_3216Metric, F.Cu at (109.9, 112.6)
- added R16: 3k3, Resistor_SMD:R_1206_3216Metric, F.Cu at (128.3, 112.6)
- added R17: 3k3, Resistor_SMD:R_1206_3216Metric, F.Cu at (146.7, 112.6)
- added R18: 3k3, Resistor_SMD:R_1206_3216Metric, F.Cu at (158.1, 115.8)
- added R7: 3k3, Resistor_SMD:R_1206_3216Metric, F.Cu at (109.9, 108.0)
- added R8: 3k3, Resistor_SMD:R_1206_3216Metric, F.Cu at (128.3, 107.8)
- added R9: 3k3, Resistor_SMD:R_1206_3216Metric, F.Cu at (146.7, 107.8)
- R5: value R -> 1k
- R6: value R -> 10k
- moved R4 9.39 mm to (157.5, 98.0), turned to 90 degrees
- moved R3 8.01 mm to (160.0, 98.0), turned to 90 degrees
- moved +5v-1 4.45 mm to (165.7, 101.0)
- moved C1 1.27 mm to (105.4, 110.2)
- moved C2 0.63 mm to (123.8, 110.2)
- moved C3 0.63 mm to (142.2, 110.2)
Routing:
- net out0: track 25.7 -> 15.9 mm
- net 5v: track 0.00 -> 9.43 mm, vias 0 -> 7
- net /driver2/step: track 9.67 -> 14.1 mm
- net /driver0/enable: track 50.5 -> 54.4 mm
- net /driver1/step: track 15.5 -> 18.9 mm
- net /driver0/step: track 35.0 -> 38.3 mm
- net /driver1/dir: track 13.8 -> 16.6 mm
- net out1: track 16.2 -> 13.4 mm
- net /driver2/dir: track 8.77 -> 11.5 mm
- net /driver0/dir: track 33.3 -> 36.0 mm
- net 12v: track 157.5 -> 154.9 mm
Other:
- board text added: "24V"
- board text added: "5V"
- board text added: "Joint1"
- board text added: "Joint2"
- board text added: "Joint3"
