File: rio-icebreaker3x.kicad_sch (KiCad schematic)
At the start: 20 parts, among them J15 Conn_02x06_Odd_Even, J16 Conn_02x06_Odd_Even, J9 Conn_01x03, Q1 BC817, U9 ULN2803A

Commit message: adding missing pullups
Parts:
- added R1: 3k3, Resistor_SMD:R_1206_3216Metric, symbol Device:R
- R1: value R -> 10k
- R1: value R -> 1k
Connections:
- net 5v: now also R1.1
- net driver0/enable: now also R1.2
Changed lines of the file:
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@@
   (junction (at 143.51 57.15) (diameter 0) (color 0 0 0 0)
   )
+  (junction (at 120.65 74.93) (diameter 0) (color 0 0 0 0)
+  )
   (junction (at 87.63 60.96) (diameter 0) (color 0 0 0 0)
   )
@@
     (stroke (width 0) (type default))
   )
-  (wire (pts (xy 120.65 66.04) (xy 120.65 78.74))
+  (wire (pts (xy 120.65 66.04) (xy 120.65 74.93))
     (stroke (width 0) (type default))
   )
@@
   )
   (wire (pts (xy 238.76 69.85) (xy 238.76 90.17))
+    (stroke (width 0) (type default))
+  )
+  (wire (pts (xy 120.65 74.93) (xy 120.65 78.74))
     (stroke (width 0) (type default))
   )
@@
     (effects (font (size 1.27 1.27)) (justify right))
     (property "Intersheetrefs" "${INTERSHEET_REFS}" (at 239.2409 25.4 0)
+      (effects (font (size 1.27 1.27)) (justify right) hide)
+    )
+  )
+  (global_label "5v" (shape input) (at 113.03 74.93 180) (fields_autoplaced)
+    (effects (font (size 1.27 1.27)) (justify right))
+    (property "Intersheetrefs" "${INTERSHEET_REFS}" (at 107.9471 74.93 0)
       (effects (font (size 1.27 1.27)) (justify right) hide)
     )
@@
         (path "/cfe43c71-4742-4fe7-be75-9d9a9d4efd01"
           (reference "R2") (unit 1)
+        )
+      )
+    )
+  )
+  (symbol (lib_id "Device:R") (at 116.84 74.93 90) (unit 1)
+    (in_bom yes) (on_board yes) (dnp no)
+    (property "Reference" "R1" (at 116.84 72.39 90)
+      (effects (font (size 1.27 1.27)))
+    )
+    (property "Value" "3k3" (at 116.84 77.47 90)
+      (effects (font (size 1.27 1.27)))
+    )
+    (property "Footprint" "Resistor_SMD:R_1206_3216Metric" (at 116.84 76.708 90)
+      (effects (font (size 1.27 1.27)) hide)
+    )
+    (property "Datasheet" "~" (at 116.84 74.93 0)
+      (effects (font (size 1.27 1.27)) hide)
+    )
+    (pin "1")
+    (pin "2")
+    (instances
+      (project "riowerks"
+        (path "/c4675d0b-5c1c-444a-a1ef-26bf66f46aa5/cda04744-3ce8-4a6b-a82d-a1325fcc2daa"
+          (reference "R1") (unit 1)
+        )
+        (path "/c4675d0b-5c1c-444a-a1ef-26bf66f46aa5/c87ea30f-b16d-4690-be9f-7e9196f340db"
+          (reference "R2") (unit 1)
+        )
+        (path "/c4675d0b-5c1c-444a-a1ef-26bf66f46aa5/0caef072-d6e6-4191-8609-a2a060f30d09"
+          (reference "R3") (unit 1)
+        )
+        (path "/c4675d0b-5c1c-444a-a1ef-26bf66f46aa5/9b7eb7c2-dba6-4078-aea0-2fd449da534f"
+          (reference "R4") (unit 1)
+        )
+        (path "/c4675d0b-5c1c-444a-a1ef-26bf66f46aa5/c4b53cc4-45b0-40c6-a2e4-f85052d4ed8a"
+          (reference "R5") (unit 1)
+        )
+        (path "/c4675d0b-5c1c-444a-a1ef-26bf66f46aa5/6dac5bea-3ac5-4905-a711-17de9963fb48"
+          (reference "R6") (unit 1)
+        )
+        (path "/c4675d0b-5c1c-444a-a1ef-26bf66f46aa5/0e9d2bbf-2b0b-4860-a06b-304bc4546dd9"
+          (reference "R7") (unit 1)
+        )
+        (path "/c4675d0b-5c1c-444a-a1ef-26bf66f46aa5/77b70234-a638-4cba-af0b-c8e26a05632f"
+          (reference "R8") (unit 1)
+        )
+        (path "/c4675d0b-5c1c-444a-a1ef-26bf66f46aa5/341fad45-713c-4626-966f-e3afd8f08c91"
+          (reference "R16") (unit 1)
+        )
+        (path "/c4675d0b-5c1c-444a-a1ef-26bf66f46aa5"
+          (reference "R43") (unit 1)
+        )
+      )
+      (project "rio-icebreaker3x"
+        (path "/cfe43c71-4742-4fe7-be75-9d9a9d4efd01"
+          (reference "R18") (unit 1)
+        )
+        (path "/cfe43c71-4742-4fe7-be75-9d9a9d4efd01/01713ad6-c8ee-4cb4-a069-0eb1e2d0d4c5"
+          (reference "R15") (unit 1)
+        )
+        (path "/cfe43c71-4742-4fe7-be75-9d9a9d4efd01/71bd7516-8b6e-4c0f-97ca-5abb746077c1"
+          (reference "R16") (unit 1)
+        )
+        (path "/cfe43c71-4742-4fe7-be75-9d9a9d4efd01/d8c46525-3323-49c5-8ba1-282344862c7d"
+          (reference "R17") (unit 1)
         )
       )
@@
   )
   (symbol (lib_id "Device:R") (at 105.41 87.63 180) (unit 1)
-    (in_bom yes) (on_board yes) (dnp no) (fields_autoplaced)
-    (property "Reference" "R1" (at 107.95 86.36 0)
+    (in_bom yes) (on_board yes) (dnp no)
+    (property "Reference" "R1" (at 101.6 87.63 0)
       (effects (font (size 1.27 1.27)) (justify right))
     )
-    (property "Value" "R" (at 107.95 88.9 0)
+    (property "Value" "10k" (at 101.6 90.17 0)
       (effects (font (size 1.27 1.27)) (justify right))
     )
@@
   )
   (symbol (lib_id "Device:R") (at 109.22 83.82 90) (unit 1)
-    (in_bom yes) (on_board yes) (dnp no) (fields_autoplaced)
-    (property "Reference" "R1" (at 109.22 77.47 90)
+    (in_bom yes) (on_board yes) (dnp no)
+    (property "Reference" "R1" (at 109.22 81.28 90)
       (effects (font (size 1.27 1.27)))
     )
-    (property "Value" "R" (at 109.22 80.01 90)
+    (property "Value" "1k" (at 109.22 86.36 90)
       (effects (font (size 1.27 1.27)))
     )
